File: nks.kicad_pcb (KiCad board)
At the start: 2 copper layers, 81 x 92 mm, 20 parts, among them J1 microSD, J2 DevKit-J1, J3 DevKit-J3, SW1 SW_SPDT, U2 RTC_DS3231+AT24C32, U3 SHT30, U4 TPS22918

Commit message: PCB completo: rutado de señales y alimentación terminado, 0 infracciones DRC (aviso de isla GND excluido)
Routing:
- net /LED_STAT: vias 2 -> 1
- net /GND: vias 0 -> 9
Changed lines of the file:
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@@
 			(net "/GND")
 			(pintype "passive")
+			(zone_connect 2)
 		)
 		(embedded_fonts no)
@@
 		(net "/BTN")
 	)
+	(via
+		(at 112 43)
+		(size 0.6)
+		(drill 0.3)
+		(layers "F.Cu" "B.Cu")
+		(free yes)
+		(net "/GND")
+	)
+	(via
+		(at 112 52)
+		(size 0.6)
+		(drill 0.3)
+		(layers "F.Cu" "B.Cu")
+		(free yes)
+		(net "/GND")
+	)
+	(via
+		(at 101 41)
+		(size 0.6)
+		(drill 0.3)
+		(layers "F.Cu" "B.Cu")
+		(net "/GND")
+	)
+	(via
+		(at 180 131)
+		(size 0.6)
+		(drill 0.3)
+		(layers "F.Cu" "B.Cu")
+		(net "/GND")
+	)
+	(via
+		(at 122 73)
+		(size 0.6)
+		(drill 0.3)
+		(layers "F.Cu" "B.Cu")
+		(net "/GND")
+	)
+	(via
+		(at 179 41)
+		(size 0.6)
+		(drill 0.3)
+		(layers "F.Cu" "B.Cu")
+		(net "/GND")
+	)
+	(via
+		(at 103 52)
+		(size 0.6)
+		(drill 0.3)
+		(layers "F.Cu" "B.Cu")
+		(free yes)
+		(net "/GND")
+	)
+	(via
+		(at 119 73)
+		(size 0.6)
+		(drill 0.3)
+		(layers "F.Cu" "B.Cu")
+		(net "/GND")
+	)
+	(via
+		(at 101 131)
+		(size 0.6)
+		(drill 0.3)
+		(layers "F.Cu" "B.Cu")
+		(net "/GND")
+	)
 	(segment
 		(start 112.3 98.7)
@@
 		(net "/LED_STAT")
 	)
-	(via
-		(at 133 61.22)
-		(size 0.6)
-		(drill 0.3)
-		(layers "F.Cu" "B.Cu")
-		(net "/LED_STAT")
-	)
 	(segment
 		(start 123 87.41)
@@
 	)
 	(segment
-		(start 142.393654 57.38)
-		(end 149.523654 64.51)
+		(start 107 54.84)
+		(end 108.39 53.45)
 		(width 0.2)
 		(layer "F.Cu")
-		(net "/I2S_SD")
+		(net "/I2S_WS")
 	)
 	(segment
-		(start 152 60.28)
-		(end 150 58.28)
+		(start 150 63.36)
+		(end 148.45 61.81)
 		(width 0.2)
 		(layer "F.Cu")
-		(net "/I2S_SD")
+		(net "/I2S_WS")
 	)
 	(segment
-		(start 149.523654 64.51)
-		(end 150.476346 64.51)
+		(start 149.523654 54.59)
+		(end 169.25 54.59)
 		(width 0.2)
 		(layer "F.Cu")
-		(net "/I2S_SD")
+		(net "/I2S_WS")
 	)
 	(segment
-		(start 152 62.986346)
-		(end 152 60.28)
+		(start 148.45 55.663654)
+		(end 149.523654 54.59)
 		(width 0.2)
 		(layer "F.Cu")
-		(net "/I2S_SD")
+		(net "/I2S_WS")
 	)
 	(segment
-		(start 150.476346 64.51)
-		(end 152 62.986346)
+		(start 107 54.84)
+		(end 107.347968 54.84)
 		(width 0.2)
 		(layer "F.Cu")
-		(net "/I2S_SD")
+		(net "/I2S_WS")
 	)
 	(segment
-		(start 150 58.28)
-		(end 170.64 58.28)
+		(start 169.25 54.59)
+		(end 170 53.84)
 		(width 0.2)
 		(layer "F.Cu")
-		(net "/I2S_SD")
+		(net "/I2S_WS")
 	)
 	(segment
-		(start 170.64 58.28)
-		(end 172.54 56.38)
+		(start 141.396546 49.51)
+		(end 146.276546 54.39)
 		(width 0.2)
 		(layer "F.Cu")
-		(net "/I2S_SD")
+		(net "/I2S_WS")
 	)
 	(segment
-		(start 109.54 57.38)
-		(end 142.393654 57.38)
+		(start 108.39 51.823654)
+		(end 110.703654 49.51)
 		(width 0.2)
 		(layer "F.Cu")
-		(net "/I2S_SD")
+		(net "/I2S_WS")
+	)
+	(segment
+		(start 110.703654 49.51)
+		(end 141.396546 49.51)
+		(width 0.2)
+		(layer "F.Cu")
+		(net "/I2S_WS")
+	)
+	(segment
+		(start 148.45 61.81)
+		(end 148.45 55.663654)
+		(width 0.2)
+		(layer "F.Cu")
+		(net "/I2S_WS")
+	)
+	(segment
+		(start 108.39 53.45)
+		(end 108.39 51.823654)
+		(width 0.2)
+		(layer "F.Cu")
+		(net "/I2S_WS")
+	)
+	(via
+		(at 146.276546 54.39)
+		(size 0.6)
+		(drill 0.3)
+		(layers "F.Cu" "B.Cu")
+		(net "/I2S_WS")
+	)
+	(segment
+		(start 146.276546 54.39)
+		(end 146.276546 59.636546)
+		(width 0.2)
+		(layer "B.Cu")
+		(net "/I2S_WS")
+	)
+	(segment
+		(start 146.276546 59.636546)
+		(end 150 63.36)
+		(width 0.2)
+		(layer "B.Cu")
+		(net "/I2S_WS")
 	)
 	(segment
@@
 	)
 	(segment
-		(start 107 54.84)
-		(end 108.39 53.45)
-		(width 0.2)
-		(layer "F.Cu")
-		(net "/I2S_WS")
-	)
-	(segment
-		(start 150 63.36)
-		(end 148.45 61.81)
-		(width 0.2)
-		(layer "F.Cu")
-		(net "/I2S_WS")
-	)
-	(segment
-		(start 149.523654 54.59)
-		(end 169.25 54.59)
-		(width 0.2)
-		(layer "F.Cu")
-		(net "/I2S_WS")
-	)
-	(segment
-		(start 148.45 55.663654)
-		(end 149.523654 54.59)
+		(start 142.393654 57.38)
+		(end 149.523654 64.51)
 		(width 0.2)
 		(layer "F.Cu")
-		(net "/I2S_WS")
+		(net "/I2S_SD")
 	)
 	(segment
-		(start 107 54.84)
-		(end 107.347968 54.84)
+		(start 152 60.28)
+		(end 150 58.28)
 		(width 0.2)
 		(layer "F.Cu")
-		(net "/I2S_WS")
+		(net "/I2S_SD")
 	)
 	(segment
-		(start 169.25 54.59)
-		(end 170 53.84)
+		(start 149.523654 64.51)
+		(end 150.476346 64.51)
 		(width 0.2)
 		(layer "F.Cu")
-		(net "/I2S_WS")
+		(net "/I2S_SD")
 	)
 	(segment
-		(start 141.396546 49.51)
-		(end 146.276546 54.39)
+		(start 152 62.986346)
+		(end 152 60.28)
 		(width 0.2)
 		(layer "F.Cu")
-		(net "/I2S_WS")
+		(net "/I2S_SD")
 	)
 	(segment
-		(start 108.39 51.823654)
-		(end 110.703654 49.51)
+		(start 150.476346 64.51)
+		(end 152 62.986346)
 		(width 0.2)
 		(layer "F.Cu")
-		(net "/I2S_WS")
+		(net "/I2S_SD")
 	)
 	(segment
-		(start 110.703654 49.51)
-		(end 141.396546 49.51)
+		(start 150 58.28)
+		(end 170.64 58.28)
 		(width 0.2)
 		(layer "F.Cu")
-		(net "/I2S_WS")
+		(net "/I2S_SD")
 	)
 	(segment
-		(start 148.45 61.81)
-		(end 148.45 55.663654)
+		(start 170.64 58.28)
+		(end 172.54 56.38)
 		(width 0.2)
 		(layer "F.Cu")
-		(net "/I2S_WS")
+		(net "/I2S_SD")
 	)
 	(segment
-		(start 108.39 53.45)
-		(end 108.39 51.823654)
+		(start 109.54 57.38)
+		(end 142.393654 57.38)
 		(width 0.2)
 		(layer "F.Cu")
-		(net "/I2S_WS")
-	)
-	(via
-		(at 146.276546 54.39)
-		(size 0.6)
-		(drill 0.3)
-		(layers "F.Cu" "B.Cu")
-		(net "/I2S_WS")
-	)
-	(segment
-		(start 146.276546 54.39)
-		(end 146.276546 59.636546)
-		(width 0.2)
-		(layer "B.Cu")
-		(net "/I2S_WS")
-	)
-	(segment
-		(start 146.276546 59.636546)
-		(end 150 63.36)
-		(width 0.2)
-		(layer "B.Cu")
-		(net "/I2S_WS")
+		(net "/I2S_SD")
 	)
 	(segment
@@
 	)
 	(segment
+		(start 118.05 73.95)
+		(end 117.1 73)
+		(width 0.2)
+		(layer "F.Cu")
+		(net "/+3V3_IN")
+	)
+	(segment
 		(start 134.01 85.47)
 		(end 129.57 85.47)
@@
 	(segment
 		(start 129.57 85.47)
-		(end 117.1 73)
+		(end 118.05 73.95)
 		(width 0.2)
 		(layer "F.Cu")
