File: nks.kicad_pcb (KiCad board)
At the start: 2 copper layers, 81 x 92 mm, 20 parts, among them J1 microSD, J2 DevKit-J1, J3 DevKit-J3, SW1 SW_SPDT, U2 RTC_DS3231+AT24C32, U3 SHT30, U4 TPS22918

Commit message: Serigrafia de montaje + texto identificativo NkS. DRC 0/0/0 limpio.
Other:
- board text added: "NkS v1.0 Nekia Systems 2026-08"
Changed lines of the file:
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@@
 		(capping no)
 		(filling no)
-		(zone_defaults)
 		(pcbplotparams
 			(layerselection 0x00000000_00000000_55555555_575555ff)
@@
 		(layer "Edge.Cuts")
 	)
+	(gr_text "NkS v1.0\nNekia Systems\n2026-08"
+		(at 164 46 0)
+		(layer "F.SilkS")
+		(effects
+			(font
+				(size 0.8 1)
+				(thickness 0.15)
+			)
+			(justify left bottom)
+		)
+	)
 	(segment
